File: hardware/dot-matrix-badge.kicad_pcb (KiCad board)
At the start: 2 copper layers, 5 parts, among them J1 AVR-ISP-6, SW1 SW_SPST, U1 ATtiny13A-SS

Commit message: cpp firmware, hardware progress
Parts:
- added H1: MountingHole, DotMatrixBadge:MountingHole_Custom, F.Cu at (30.2, 32.2)
- added H2: MountingHole, DotMatrixBadge:MountingHole_Custom, F.Cu at (30.2, 47.7)
- added H3: MountingHole, DotMatrixBadge:MountingHole_Custom, F.Cu at (84.9, 32.1)
- added H4: MountingHole, DotMatrixBadge:MountingHole_Custom, F.Cu at (84.8, 47.9)
- BT1: footprint Battery:BatteryHolder_Multicomp_BC-2001_1x2032 -> Battery:BatteryHolder_Keystone_3034_1x20mm
- D1: footprint HCMS-291x:HCMS-291X -> DotMatrixBadge:HCMS-291X
- J1: value AVR-ISP-6 -> AVR-UPDI-6; footprint Connector_PinSocket_2.54mm:PinSocket_2x03_P2.54mm_Vertical -> DotMatrixBadge:UPDI_Pads
- SW1: moved to B.Cu
- U1: value ATtiny13A-SS -> ATtiny402-SS
- moved SW1 48.1 mm to (59.5, 48.0), turned to 180 degrees
- moved D1 39.5 mm to (48.0, 40.0)
- moved U1 39.0 mm to (75.0, 40.0), turned to -90 degrees
- moved J1 30.1 mm to (47.5, 48.0)
- moved BT1 25.0 mm to (75.0, 40.1)
Connections:
- D1 pad 15: MISO/RS -> RS
- D1 pad 17: SCK/CLK -> CLK
- D1 pad 19: MOSI/BLANK -> BL
- J1 pad 1: MISO/RS -> UPDI
- U1 pad 1: RST -> +3V3
- U1 pad 2: CE -> CLK
- U1 pad 3: DIN -> RS
- U1 pad 4: GND -> DIN
- U1 pad 5: MOSI/BLANK -> BL
- U1 pad 6: MISO/RS -> UPDI
- U1 pad 7: SCK/CLK -> CE
- U1 pad 8: +3V3 -> GND
Routing:
- net +3V3: track 0.00 -> 64.4 mm
- net GND: track 0.00 -> 62.9 mm
- net BL: track 0.00 -> 48.3 mm
- net CE: track 0.00 -> 40.2 mm
- net UPDI: track 0.00 -> 25.1 mm
- net CLK: track 0.00 -> 24.0 mm
- net RS: track 0.00 -> 17.0 mm
- net DIN: track 0.00 -> 12.6 mm
Other:
- board outline added: 59 x 20 mm

Commit message: almost done with layout
Parts:
- added SW2: SW_Push, DotMatrixBadge:SW_SPST_PTS526_JLeads, F.Cu at (69.0, 45.0)
- added SW3: SW_Push, DotMatrixBadge:SW_SPST_PTS526_JLeads, F.Cu at (75.8, 45.0)
- U1: value ATtiny402-SS -> ATtiny1604-SS; footprint Package_SO:SOIC-8_3.9x4.9mm_P1.27mm -> Package_SO:SOIC-14_3.9x8.7mm_P1.27mm
- moved SW1 20.6 mm to (38.9, 47.9)
- moved J1 17.0 mm to (41.4, 32.1)
- moved U1 4.01 mm to (72.4, 37.0)
- moved H3 4.00 mm to (80.9, 32.1)
- moved H4 4.00 mm to (80.8, 47.9)
- moved BT1 3.93 mm to (71.1, 40.1)
- moved D1 1.47 mm to (46.5, 40.0)
Connections:
- D1 pad 10: +3V3 -> VCC
- D1 pad 21: +3V3 -> VCC
- D1 pad 22: +3V3 -> VCC
- D1 pad 25: unconnected-(D1-OSC-Pad25) -> OSC
- D1 pad 26: unconnected-(D1-DOUT-Pad26) -> DOUT
- D1 pad 3: +3V3 -> VCC
- J1 pad 2: +3V3 -> VCC
- SW1 pad 1: +3V3 -> Net-(BT1-+)
- SW1 pad 2: Net-(BT1-+) -> VCC
- U1 pad 1: +3V3 -> VCC
- U1 pad 2: CLK -> DOUT
- U1 pad 3: RS -> OSC
- U1 pad 4: DIN -> BL
- U1 pad 5: BL -> CLK
- U1 pad 6: UPDI -> CE
- U1 pad 7: CE -> GND
Routing:
- net VCC: track 0.00 -> 216.3 mm
- net GND: track 62.9 -> 193.7 mm
- net +3V3: track 64.4 -> 0.00 mm
- net DOUT: track 0.00 -> 52.8 mm
- net OSC: track 0.00 -> 47.4 mm
- net Net-(BT1-+): track 0.00 -> 34.1 mm
- net BL: track 48.3 -> 29.2 mm
- net CE: track 40.2 -> 24.0 mm
- net BTN1: track 0.00 -> 15.4 mm
- net UPDI: track 25.1 -> 40.5 mm, vias 0 -> 1
- net BTN2: track 0.00 -> 9.09 mm
- net RS: track 17.0 -> 13.9 mm
- net CLK: track 24.0 -> 22.7 mm
- net DIN: track 12.6 -> 13.8 mm
Other:
- board size 59 x 20 mm -> 55 x 20 mm

Commit message: pcb payout almost complete
Parts:
- added BT2: Battery_Cell, DotMatrixBadge:SpareBatteryHolder_Keystone_3034_1x20mm, B.Cu at (54.8, 28.7)
- added D2: LED, LED_SMD:LED_0603_1608Metric, F.Cu at (75.7, 37.3)
- added J2: JST_04, Connector_JST:JST_SH_BM04B-SRSS-TB_1x04-1MP_P1.00mm_Vertical, B.Cu at (70.4, 20.0)
- added R1: 1k, Resistor_SMD:R_0402_1005Metric, F.Cu at (70.4, 37.0)
- moved SW1 33.2 mm to (70.4, 37.5)
- moved H1 19.4 mm to (45.1, 19.8)
- moved H3 19.4 mm to (95.8, 19.7)
- moved BT1 18.7 mm to (86.0, 28.7)
- moved D1 18.7 mm to (61.4, 28.6)
- moved U1 18.7 mm to (87.3, 25.6), turned to 90 degrees
- moved SW2 18.6 mm to (83.8, 33.9)
- moved SW3 18.6 mm to (90.7, 33.9)
- moved H4 18.1 mm to (95.7, 37.5)
- moved H2 18.1 mm to (45.1, 37.4)
- moved J1 16.1 mm to (51.2, 19.3), turned to 0 degrees
Connections:
- D1 pad 24: GND -> RESET
- U1 pad 11: DIN -> BL
- U1 pad 12: BTN1 -> CLK
- U1 pad 13: BTN2 -> CE
- U1 pad 2: DOUT -> RS
- U1 pad 4: BL -> DIN
- U1 pad 5: CLK -> BTN1
- U1 pad 6: CE -> BTN2
- U1 pad 7: GND -> SCL
- U1 pad 8: GND -> SDA
- U1 pad 9: RS -> RESET
Routing:
- net VCC: track 216.3 -> 149.6 mm, vias 0 -> 1
- net SDA: track 0.00 -> 64.9 mm, vias 0 -> 1
- net RESET: track 0.00 -> 54.9 mm
- net SCL: track 0.00 -> 45.5 mm, vias 0 -> 1
- net DOUT: track 52.8 -> 86.7 mm
- net UPDI: track 40.5 -> 63.9 mm
- net OSC: track 47.4 -> 62.9 mm
- net Net-(BT1-+): track 34.1 -> 45.8 mm
- net Net-(D2-A): track 0.00 -> 11.5 mm
- net GND: track 193.7 -> 198.0 mm, vias 0 -> 2
- net RS: track 13.9 -> 16.9 mm
- net CLK: track 22.7 -> 24.0 mm
- net DIN: track 13.8 -> 14.9 mm
- net CE: track 24.0 -> 25.0 mm
- net BL: track 29.2 -> 30.0 mm
Other:
- board size 55 x 20 mm -> 55 x 22 mm

Commit message: 99% done
Parts:
- R1: footprint Resistor_SMD:R_0402_1005Metric -> Resistor_SMD:R_0603_1608Metric
- moved R1 0.43 mm to (70.4, 37.4)
- moved D1 0.05 mm to (75.7, 37.4)
- renumbered D2 to D1
Routing:
- net VCC: track 149.6 -> 204.8 mm
- net SCL: track 45.5 -> 71.0 mm
- net SDA: track 64.9 -> 86.7 mm, vias 1 -> 0
- net DIN: track 14.9 -> 27.5 mm
- net GND: track 198.0 -> 207.4 mm
- net DOUT: track 86.7 -> 91.3 mm
- net UPDI: track 63.9 -> 59.9 mm, vias 1 -> 0
- net Net-(D2-A): track 11.5 -> 10.7 mm

Commit message: halfway through symbol/footprint cleanup
Parts:
- added J3: Test Pads, DotMatrixBadge:Pads_1x5_1mm, F.Cu at (95.8, 28.6)
- J2: value JST_04 -> Qwiic/Stemma QT; footprint Connector_JST:JST_SH_BM04B-SRSS-TB_1x04-1MP_P1.00mm_Vertical -> DotMatrixBadge:JST_SH_4P_No Silkscreen
- renumbered D1 to U1, U1 to U2
Routing:
- net VCC: track 204.8 -> 195.6 mm
- net SCL: track 71.0 -> 63.6 mm
- net SDA: track 86.7 -> 90.7 mm
- net DIN: track 27.5 -> 30.7 mm
- net UPDI: track 59.9 -> 62.0 mm, vias 0 -> 1

Commit message: done with cleanup, making things pretty
Parts:
- BT1: footprint Battery:BatteryHolder_Keystone_3034_1x20mm -> DotMatrixBadge:BatteryHolder_Keystone_3034_1x20mm
- D1: footprint LED_SMD:LED_0603_1608Metric -> DotMatrixBadge:LED_0603_1608Metric
- R1: footprint Resistor_SMD:R_0603_1608Metric -> DotMatrixBadge:R_0603_1608Metric
- SW1: footprint Button_Switch_SMD:SW_SPDT_PCM12 -> DotMatrixBadge:SW_SPDT_PCM12
- U2: footprint Package_SO:SOIC-14_3.9x8.7mm_P1.27mm -> DotMatrixBadge:SOIC-14_3.9x8.7mm_P1.27mm
- moved J2 0.10 mm to (70.4, 20.1)
- moved BT2 0.07 mm to (54.9, 28.7)
- moved BT1 0.07 mm to (85.9, 28.7)
Connections:
- U2 pad 12: CLK -> CE
- U2 pad 13: CE -> CLK
Routing:
- net GND: track 207.6 -> 250.5 mm, vias 2 -> 0
- net RESET: track 54.9 -> 69.6 mm
- net DOUT: track 91.6 -> 81.8 mm
- net VCC: track 195.6 -> 187.1 mm
- net OSC: track 62.9 -> 56.2 mm
- net CE: track 25.0 -> 30.8 mm
- net DIN: track 30.7 -> 28.0 mm
- net UPDI: track 62.0 -> 59.6 mm
- net SCL: track 63.6 -> 61.6 mm
- net SDA: track 90.7 -> 88.8 mm, vias 0 -> 1
- net CLK: track 24.0 -> 22.4 mm
Other:
- rule pad_to_mask_clearance: 0 -> 0.0508
