File: hardware/dot-matrix-badge.kicad_sch (KiCad schematic)
At the start: 5 parts, among them J1 AVR-ISP-6, SW1 SW_SPST, U1 ATtiny13A-SS

Commit message: cpp firmware, hardware progress
Parts:
- removed J1: AVR-ISP-6, Connector_PinSocket_2.54mm:PinSocket_2x03_P2.54mm_Vertical, symbol Connector:AVR-ISP-6
- removed U1: ATtiny13A-SS, Package_SO:SOIC-8_3.9x4.9mm_P1.27mm, symbol MCU_Microchip_ATtiny:ATtiny13A-SS
- added H1, H2, H3, H4: MountingHole, DotMatrixBadge:MountingHole_Custom, symbol Mechanical:MountingHole
- added J1: AVR-UPDI-6, DotMatrixBadge:UPDI_Pads, symbol Connector:AVR-UPDI-6
- added U1: ATtiny402-SS, Package_SO:SOIC-8_3.9x4.9mm_P1.27mm, symbol MCU_Microchip_ATtiny:ATtiny402-SS
- BT1: footprint Battery:BatteryHolder_Multicomp_BC-2001_1x2032 -> Battery:BatteryHolder_Keystone_3034_1x20mm
- D1: footprint HCMS-291x:HCMS-291X -> DotMatrixBadge:HCMS-291X; symbol HCMS-291X:HCMS-291X -> DotMatrixBadge:HCMS-291X
Connections:
- net +3V3: now also J1.2 (VCC), U1.1 (VCC)
- net CE: now also U1.7 (PA3)
- net DIN: now also U1.4 (PA1)
- net GND: now also J1.6 (GND), U1.8 (GND)
- net MISO/RS renamed RS
- net RS: now also U1.3 (PA7)
- net MOSI/BLANK renamed BL
- net BL: now also U1.5 (PA2)
- net SCK/CLK renamed CLK
- net CLK: now also U1.2 (PA6)
- new net UPDI: J1.1 (DATA), U1.6 (~{RESET}/PA0)
Other:
- moved on the sheet: BT1, D1, SW1

Commit message: almost done with layout
Parts:
- removed U1: ATtiny402-SS, Package_SO:SOIC-8_3.9x4.9mm_P1.27mm, symbol MCU_Microchip_ATtiny:ATtiny402-SS
- added SW2, SW3: SW_Push, DotMatrixBadge:SW_SPST_PTS526_JLeads, symbol Switch:SW_Push
- added U1: ATtiny1604-SS, Package_SO:SOIC-14_3.9x8.7mm_P1.27mm, symbol MCU_Microchip_ATtiny:ATtiny1604-SS
Connections:
- net +3V3: no longer D1.10 (V_LED), D1.21 (SEL), D1.22 (V_LOGIC), D1.3 (V_LED), J1.2 (VCC), SW1.1 (A)
- net BL: now also U1.4 (PA6)
- net CE: now also U1.6 (PB3)
- net CLK: now also U1.5 (PA7)
- net DIN: now also U1.11 (PA1)
- net GND: now also SW2.2, SW3.2, U1.14 (GND), U1.7 (PB2), U1.8 (PB1)
- net RS: now also U1.9 (PB0)
- net UPDI: now also U1.10 (~{RESET}/PA0)
- net at BT1.1 (+): now also SW1.1 (A); no longer SW1.2 (B)
- net OSC: now reaches D1.25 (OSC)
- net OSC: now also U1.3 (PA5)
- net DOUT: now reaches D1.26 (DOUT)
- net DOUT: now also U1.2 (PA4)
- new net BTN1: SW2.1, U1.12 (PA2)
- new net BTN2: SW3.1, U1.13 (PA3)
- new net VCC: D1.10 (V_LED), D1.21 (SEL), D1.22 (V_LOGIC), D1.3 (V_LED), J1.2 (VCC), SW1.2 (B), U1.1 (VCC)
- no-connect marks 2 -> 0
Other:
- moved on the sheet: BT1, H1, H2, H3, H4, J1, SW1

Commit message: pcb payout almost complete
Parts:
- added BT2: Battery_Cell, DotMatrixBadge:SpareBatteryHolder_Keystone_3034_1x20mm, symbol Device:Battery_Cell
- added D2: LED, LED_SMD:LED_0603_1608Metric, symbol Device:LED
- added J2: JST_04, Connector_JST:JST_SH_BM04B-SRSS-TB_1x04-1MP_P1.00mm_Vertical, symbol PCM_SL_Connectors:JST_04
- added R1: 1k, Resistor_SMD:R_0402_1005Metric, symbol PCM_SL_Resistors:Resistor
Connections:
- net BL: now also U1.11 (PA1); no longer U1.4 (PA6)
- net BTN1: now also U1.5 (PA7); no longer U1.12 (PA2)
- net BTN2: now also U1.6 (PB3); no longer U1.13 (PA3)
- net CE: now also U1.13 (PA3); no longer U1.6 (PB3)
- net CLK: now also U1.12 (PA2); no longer U1.5 (PA7)
- net DIN: now also U1.4 (PA6); no longer U1.11 (PA1)
- net DOUT: now also R1.2; no longer U1.2 (PA4)
- net GND: now also D2.1 (K), J2.4; no longer D1.24 (~{RESET}), U1.7 (PB2), U1.8 (PB1)
- net RS: now also U1.2 (PA4); no longer U1.9 (PB0)
- net VCC: now also J2.3
- new net: D2.2 (A), R1.1
- new net RESET: D1.24 (~{RESET}), U1.9 (PB0)
- new net SCL: J2.1, U1.7 (PB2)
- new net SDA: J2.2, U1.8 (PB1)
- no-connect marks 0 -> 2
Other:
- moved on the sheet: BT1, D1, H1, H2, H3, H4, J1, SW1, SW2, SW3, U1

Commit message: 99% done
Parts:
- added J3: Test Pads, symbol Connector:Conn_01x05_Pin
- J1: symbol Connector:AVR-UPDI-6 -> DotMatrixBadge:AVR-UPDI-3
- J2: value JST_04 -> Qwiic/Stemma QT
- R1: footprint Resistor_SMD:R_0402_1005Metric -> Resistor_SMD:R_0603_1608Metric
- renumbered D2 to D1
Connections:
- net DIN: now also J3.1 (Pin_1)
- net GND: now also J1.3 (GND), J3.5 (Pin_5); no longer J1.6 (GND)
- net SCL: now also J3.2 (Pin_2)
- net SDA: now also J3.3 (Pin_3)
- net VCC: now also J3.4 (Pin_4)
Other:
- note added: "Buttons"
- note added: "Connectors/Pads"
- note added: "Dot Matrix"
- note added: "LED"
- note added: "MCU"
- note added: "Mounting Holes"
- note added: "Power"
- title: (none) -> Dot Matrix Badge
- moved on the sheet: BT1, BT2, D1, H1, H2, H3, H4, J2, R1, SW1, SW2, SW3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

Commit message: halfway through symbol/footprint cleanup
Parts:
- BT2: symbol Device:Battery_Cell -> DotMatrixBadge:Battery_Cell_Spare
- J2: footprint Connector_JST:JST_SH_BM04B-SRSS-TB_1x04-1MP_P1.00mm_Vertical -> DotMatrixBadge:JST_SH_4P_No Silkscreen; symbol PCM_SL_Connectors:JST_04 -> DotMatrixBadge:JST_04_Fixed
- J3: footprint (none) -> DotMatrixBadge:Pads_1x5_1mm
- renumbered D1 to U1, U1 to U2
Connections:
- net GND: now also J3.4 (Pin_4); no longer J3.5 (Pin_5)
- net VCC: now also J3.5 (Pin_5); no longer J3.4 (Pin_4)
Changed lines of the file:
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@@
 	(wire
 		(pts
+			(xy 147.32 62.23) (xy 149.86 62.23)
+		)
+		(stroke
+			(width 0)
+			(type default)
+		)
+	)
+	(wire
+		(pts
 			(xy 67.31 24.13) (xy 67.31 25.4)
 		)
@@
 	(wire
 		(pts
+			(xy 147.32 69.85) (xy 149.86 69.85)
+		)
+		(stroke
+			(width 0)
+			(type default)
+		)
+	)
+	(wire
+		(pts
 			(xy 152.4 31.75) (xy 143.51 31.75)
 		)
@@
 	(wire
 		(pts
-			(xy 149.86 63.5) (xy 149.86 64.77)
+			(xy 149.86 62.23) (xy 149.86 64.77)
 		)
 		(stroke
@@
 	(wire
 		(pts
-			(xy 149.86 67.31) (xy 149.86 68.58)
+			(xy 149.86 67.31) (xy 149.86 69.85)
 		)
 		(stroke
@@
 	)
 	(symbol
-		(lib_id "PCM_SL_Connectors:JST_04")
+		(lib_id "DotMatrixBadge:JST_04_Fixed")
 		(at 161.29 44.45 0)
 		(unit 1)
@@
 			)
 		)
-		(property "Footprint" "Connector_JST:JST_SH_BM04B-SRSS-TB_1x04-1MP_P1.00mm_Vertical"
+		(property "Footprint" "DotMatrixBadge:JST_SH_4P_No Silkscreen"
 			(at 161.29 35.306 0)
 			(effects
@@
 	)
 	(symbol
-		(lib_id "power:GND")
-		(at 149.86 68.58 0)
-		(mirror y)
-		(unit 1)
-		(exclude_from_sim no)
-		(in_bom yes)
-		(on_board yes)
-		(dnp no)
-		(property "Reference" "#PWR015"
-			(at 149.86 74.93 0)
-			(effects
-				(font
-					(size 1.27 1.27)
-				)
-				(hide yes)
-			)
-		)
-		(property "Value" "GND"
-			(at 147.574 68.58 0)
-			(effects
-				(font
-					(size 1.27 1.27)
-				)
-			)
-		)
-		(property "Footprint" ""
-			(at 149.86 68.58 0)
-			(effects
-				(font
-					(size 1.27 1.27)
-				)
-				(hide yes)
-			)
-		)
-		(property "Datasheet" ""
-			(at 149.86 68.58 0)
-			(effects
-				(font
-					(size 1.27 1.27)
-				)
-				(hide yes)
-			)
-		)
-		(property "Description" "Power symbol creates a global label with name \"GND\" , ground"
-			(at 149.86 68.58 0)
-			(effects
-				(font
-					(size 1.27 1.27)
-				)
-				(hide yes)
-			)
-		)
-		(pin "1"
-		)
-		(instances
-			(project "dot-matrix-badge"
-				(path "/1b540e36-998f-4dd7-90ae-747ee59fea59"
-					(reference "#PWR015")
-					(unit 1)
-				)
-			)
-		)
-	)
-	(symbol
 		(lib_id "Connector:Conn_01x05_Pin")
 		(at 162.56 62.23 0)
@@
 			)
 		)
-		(property "Footprint" ""
+		(property "Footprint" "DotMatrixBadge:Pads_1x5_1mm"
 			(at 162.56 62.23 0)
 			(effects
@@
 		(dnp no)
 		(fields_autoplaced yes)
-		(property "Reference" "D1"
+		(property "Reference" "U1"
 			(at 48.26 17.78 0)
 			(effects
@@
 			(project ""
 				(path "/1b540e36-998f-4dd7-90ae-747ee59fea59"
-					(reference "D1")
+					(reference "U1")
 					(unit 1)
 				)
@@
 	)
 	(symbol
-		(lib_id "Device:Battery_Cell")
+		(lib_id "DotMatrixBadge:Battery_Cell_Spare")
 		(at 62.23 107.95 0)
 		(unit 1)
@@
 	)
 	(symbol
-		(lib_id "power:+3V3")
-		(at 149.86 63.5 0)
+		(lib_id "Mechanical:MountingHole")
+		(at 153.67 97.79 0)
 		(unit 1)
-		(exclude_from_sim no)
-		(in_bom yes)
+		(exclude_from_sim yes)
+		(in_bom no)
 		(on_board yes)
 		(dnp no)
-		(property "Reference" "#PWR018"
-			(at 149.86 67.31 0)
+		(fields_autoplaced yes)
+		(property "Reference" "H2"
+			(at 156.21 96.5199 0)
 			(effects
 				(font
 					(size 1.27 1.27)
 				)
-				(hide yes)
+				(justify left)
 			)
 		)
-		(property "Value" "VCC"
-			(at 145.542 63.754 0)
+		(property "Value" "MountingHole"
+			(at 156.21 99.0599 0)
 			(effects
 				(font
@@
 			)
 		)
-		(property "Footprint" ""
-			(at 149.86 63.5 0)
+		(property "Footprint" "DotMatrixBadge:MountingHole_Custom"
+			(at 153.67 97.79 0)
 			(effects
 				(font
@@
 			)
 		)
-		(property "Datasheet" ""
-			(at 149.86 63.5 0)
+		(property "Datasheet" "~"
+			(at 153.67 97.79 0)
 			(effects
 				(font
@@
 			)
 		)
-		(property "Description" "Power symbol creates a global label with name \"+3V3\""
-			(at 149.86 63.5 0)
+		(property "Description" "Mounting Hole without connection"
+			(at 153.67 97.79 0)
 			(effects
 				(font
@@
 			)
 		)
-		(pin "1"
-		)
 		(instances
 			(project "dot-matrix-badge"
 				(path "/1b540e36-998f-4dd7-90ae-747ee59fea59"
-					(reference "#PWR018")
+					(reference "H2")
 					(unit 1)
 				)
@@
 	)
 	(symbol
-		(lib_id "Mechanical:MountingHole")
-		(at 153.67 97.79 0)
+		(lib_id "power:GND")
+		(at 147.32 62.23 0)
+		(mirror y)
 		(unit 1)
-		(exclude_from_sim yes)
-		(in_bom no)
+		(exclude_from_sim no)
+		(in_bom yes)
 		(on_board yes)
 		(dnp no)
-		(fields_autoplaced yes)
-		(property "Reference" "H2"
-			(at 156.21 96.5199 0)
+		(property "Reference" "#PWR015"
+			(at 147.32 68.58 0)
 			(effects
 				(font
 					(size 1.27 1.27)
 				)
-				(justify left)
+				(hide yes)
 			)
 		)
-		(property "Value" "MountingHole"
-			(at 156.21 99.0599 0)
+		(property "Value" "GND"
+			(at 145.034 62.23 0)
 			(effects
 				(font
 					(size 1.27 1.27)
 				)
-				(justify left)
 			)
 		)
-		(property "Footprint" "DotMatrixBadge:MountingHole_Custom"
-			(at 153.67 97.79 0)
+		(property "Footprint" ""
+			(at 147.32 62.23 0)
 			(effects
 				(font
@@
 			)
 		)
-		(property "Datasheet" "~"
-			(at 153.67 97.79 0)
+		(property "Datasheet" ""
+			(at 147.32 62.23 0)
 			(effects
 				(font
@@
 			)
 		)
-		(property "Description" "Mounting Hole without connection"
-			(at 153.67 97.79 0)
+		(property "Description" "Power symbol creates a global label with name \"GND\" , ground"
+			(at 147.32 62.23 0)
 			(effects
 				(font
@@
 			)
 		)
+		(pin "1"
+		)
 		(instances
 			(project "dot-matrix-badge"
 				(path "/1b540e36-998f-4dd7-90ae-747ee59fea59"
-					(reference "H2")
+					(reference "#PWR015")
 					(unit 1)
 				)
@@
 	)
 	(symbol
+		(lib_id "power:+3V3")
+		(at 147.32 69.85 0)
+		(unit 1)
+		(exclude_from_sim no)
+		(in_bom yes)
+		(on_board yes)
+		(dnp no)
+		(property "Reference" "#PWR018"
+			(at 147.32 73.66 0)
+			(effects
+				(font
+					(size 1.27 1.27)
+				)
+				(hide yes)
+			)
+		)
+		(property "Value" "VCC"
+			(at 143.002 70.104 0)
+			(effects
+				(font
+					(size 1.27 1.27)
+				)
+				(justify left)
+			)
+		)
+		(property "Footprint" ""
+			(at 147.32 69.85 0)
+			(effects
+				(font
+					(size 1.27 1.27)
+				)
+				(hide yes)
+			)
+		)
+		(property "Datasheet" ""
+			(at 147.32 69.85 0)
+			(effects
+				(font
+					(size 1.27 1.27)
+				)
+				(hide yes)
+			)
+		)
+		(property "Description" "Power symbol creates a global label with name \"+3V3\""
+			(at 147.32 69.85 0)
+			(effects
+				(font
+					(size 1.27 1.27)
+				)
+				(hide yes)
+			)
+		)
+		(pin "1"
+		)
+		(instances
+			(project "dot-matrix-badge"
+				(path "/1b540e36-998f-4dd7-90ae-747ee59fea59"
+					(reference "#PWR018")
+					(unit 1)
+				)
+			)
+		)
+	)
+	(symbol
 		(lib_id "power:GND")
 		(at 104.14 58.42 0)
@@
 		(dnp no)
 		(fields_autoplaced yes)
-		(property "Reference" "U1"
+		(property "Reference" "U2"
 			(at 106.3341 20.32 0)
 			(effects
@@
 			(project ""
 				(path "/1b540e36-998f-4dd7-90ae-747ee59fea59"
-					(reference "U1")
+					(reference "U2")
 					(unit 1)
 				)

Commit message: done with cleanup, making things pretty
Parts:
- BT1: footprint Battery:BatteryHolder_Keystone_3034_1x20mm -> DotMatrixBadge:BatteryHolder_Keystone_3034_1x20mm
- D1: footprint LED_SMD:LED_0603_1608Metric -> DotMatrixBadge:LED_0603_1608Metric
- R1: footprint Resistor_SMD:R_0603_1608Metric -> DotMatrixBadge:R_0603_1608Metric
- SW1: footprint Button_Switch_SMD:SW_SPDT_PCM12 -> DotMatrixBadge:SW_SPDT_PCM12
- U2: footprint Package_SO:SOIC-14_3.9x8.7mm_P1.27mm -> DotMatrixBadge:SOIC-14_3.9x8.7mm_P1.27mm
Connections:
- net CE: now also U2.12 (PA2); no longer U2.13 (PA3)
- net CLK: now also U2.13 (PA3); no longer U2.12 (PA2)
Changed lines of the file:
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@@
+	(global_label "CE"
+		(shape input)
+		(at 119.38 35.56 0)
+		(fields_autoplaced yes)
+		(effects
+			(font
+				(size 1.27 1.27)
+			)
+			(justify left)
+		)
+		(property "Intersheetrefs" "${INTERSHEET_REFS}"
+			(at 124.7842 35.56 0)
+			(effects
+				(font
+					(size 1.27 1.27)
+				)
+				(justify left)
+				(hide yes)
+			)
+		)
+	)
 	(global_label "CE"
 		(shape input)
@@
 		)
 	)
-	(global_label "CLK"
+	(global_label "OSC"
 		(shape input)
-		(at 119.38 35.56 0)
+		(at 119.38 43.18 0)
 		(fields_autoplaced yes)
 		(effects
@@
 		)
 		(property "Intersheetrefs" "${INTERSHEET_REFS}"
-			(at 125.9333 35.56 0)
-			(effects
-				(font
-					(size 1.27 1.27)
-				)
-				(justify left)
-				(hide yes)
-			)
-		)
-	)
-	(global_label "OSC"
+			(at 126.1752 43.18 0)
+			(effects
+				(font
+					(size 1.27 1.27)
+				)
+				(justify left)
+				(hide yes)
+			)
+		)
+	)
+	(global_label "CLK"
 		(shape input)
-		(at 119.38 43.18 0)
+		(at 119.38 38.1 0)
 		(fields_autoplaced yes)
 		(effects
@@
 		)
 		(property "Intersheetrefs" "${INTERSHEET_REFS}"
-			(at 126.1752 43.18 0)
+			(at 125.9333 38.1 0)
 			(effects
 				(font
@@
 		)
 	)
-	(global_label "CE"
+	(global_label "BL"
 		(shape input)
-		(at 119.38 38.1 0)
+		(at 119.38 33.02 0)
 		(fields_autoplaced yes)
 		(effects
@@
 		)
 		(property "Intersheetrefs" "${INTERSHEET_REFS}"
-			(at 124.7842 38.1 0)
-			(effects
-				(font
-					(size 1.27 1.27)
-				)
-				(justify left)
-				(hide yes)
-			)
-		)
-	)
-	(global_label "BL"
+			(at 124.6633 33.02 0)
+			(effects
+				(font
+					(size 1.27 1.27)
+				)
+				(justify left)
+				(hide yes)
+			)
+		)
+	)
+	(global_label "SCL"
 		(shape input)
-		(at 119.38 33.02 0)
+		(at 156.21 40.64 180)
 		(fields_autoplaced yes)
 		(effects
@@
 				(size 1.27 1.27)
 			)
-			(justify left)
+			(justify right)
 		)
 		(property "Intersheetrefs" "${INTERSHEET_REFS}"
-			(at 124.6633 33.02 0)
-			(effects
-				(font
-					(size 1.27 1.27)
-				)
-				(justify left)
+			(at 149.7172 40.64 0)
+			(effects
+				(font
+					(size 1.27 1.27)
+				)
+				(justify right)
 				(hide yes)
 			)
@@
 	(global_label "SCL"
 		(shape input)
-		(at 156.21 40.64 180)
+		(at 157.48 59.69 180)
 		(fields_autoplaced yes)
 		(effects
@@
 		)
 		(property "Intersheetrefs" "${INTERSHEET_REFS}"
-			(at 149.7172 40.64 0)
+			(at 150.9872 59.69 0)
 			(effects
 				(font
@@
 		)
 	)
-	(global_label "SCL"
+	(global_label "DOUT"
 		(shape input)
-		(at 157.48 59.69 180)
+		(at 30.48 60.96 180)
 		(fields_autoplaced yes)
 		(effects
@@
 		)
 		(property "Intersheetrefs" "${INTERSHEET_REFS}"
-			(at 150.9872 59.69 0)
+			(at 22.5962 60.96 0)
 			(effects
 				(font
@@
 		)
 	)
-	(global_label "DOUT"
+	(global_label "SDA"
 		(shape input)
-		(at 30.48 60.96 180)
+		(at 88.9 33.02 180)
 		(fields_autoplaced yes)
 		(effects
@@
 		)
 		(property "Intersheetrefs" "${INTERSHEET_REFS}"
-			(at 22.5962 60.96 0)
+			(at 82.3467 33.02 0)
 			(effects
 				(font
@@
 		)
 	)
-	(global_label "SDA"
+	(global_label "UPDI"
 		(shape input)
-		(at 88.9 33.02 180)
+		(at 152.4 26.67 180)
 		(fields_autoplaced yes)
 		(effects
@@
 		)
 		(property "Intersheetrefs" "${INTERSHEET_REFS}"
-			(at 82.3467 33.02 0)
+			(at 144.9395 26.67 0)
 			(effects
 				(font
@@
 		)
 	)
-	(global_label "UPDI"
+	(global_label "SDA"
 		(shape input)
-		(at 152.4 26.67 180)
+		(at 157.48 62.23 180)
 		(fields_autoplaced yes)
 		(effects
@@
 		)
 		(property "Intersheetrefs" "${INTERSHEET_REFS}"
-			(at 144.9395 26.67 0)
-			(effects
-				(font
-					(size 1.27 1.27)
-				)
-				(justify right)
-				(hide yes)
-			)
-		)
-	)
-	(global_label "SDA"
-		(shape input)
-		(at 157.48 62.23 180)
-		(fields_autoplaced yes)
-		(effects
-			(font
-				(size 1.27 1.27)
-			)
-			(justify right)
-		)
-		(property "Intersheetrefs" "${INTERSHEET_REFS}"
 			(at 150.9267 62.23 0)
 			(effects
@@
 			)
 		)
-		(property "Footprint" "LED_SMD:LED_0603_1608Metric"
+		(property "Footprint" "DotMatrixBadge:LED_0603_1608Metric"
 			(at 118.11 110.49 0)
 			(effects
@@
 			)
 		)
-		(property "Footprint" "Button_Switch_SMD:SW_SPDT_PCM12"
+		(property "Footprint" "DotMatrixBadge:SW_SPDT_PCM12"
 			(at 48.26 97.79 0)
 			(effects
@@
 			)
 		)
-		(property "Footprint" "Resistor_SMD:R_0603_1608Metric"
+		(property "Footprint" "DotMatrixBadge:R_0603_1608Metric"
 			(at 109.601 106.172 0)
 			(effects
@@
 			)
 		)
-		(property "Footprint" "Battery:BatteryHolder_Keystone_3034_1x20mm"
+		(property "Footprint" "DotMatrixBadge:BatteryHolder_Keystone_3034_1x20mm"
 			(at 48.26 106.426 90)
 			(effects
@@
 			)
 		)
-		(property "Footprint" "Package_SO:SOIC-14_3.9x8.7mm_P1.27mm"
+		(property "Footprint" "DotMatrixBadge:SOIC-14_3.9x8.7mm_P1.27mm"
 			(at 104.14 40.64 0)
 			(effects
