File: hardware/kicad8.0/NONIK0.kicad_pcb (KiCad board)
At the start: 2 copper layers, 55 x 22 mm, 16 parts, among them J1 AVR-UPDI-6, J2 Qwiic/Stemma QT, J3 Test Pads, SW1 SW_SPST, SW2 SW_Push, SW3 SW_Push, U1 HCMS-291X, U2 ATtiny1604-SS

Commit message: buzzer
Parts:
- added BZ1: Buzzer, NONIK0:CMT-322-65-SMT-TR, F.Cu at (50.0, 20.0)
- added R2: 1K, NONIK0:R_0603_1608Metric, F.Cu at (50.5, 41.0)
Connections:
- U1 pad 25: OSC -> GND
- U2 pad 3: OSC -> BUZZ
Routing:
- net OSC: track 56.2 -> 0.00 mm
- net BUZZ: track 0.00 -> 38.3 mm
- net VCC: track 187.1 -> 160.1 mm
- net RESET: track 69.6 -> 52.1 mm

Commit message: adding power reg and piezo
Parts:
- added C1: 10u, NONIK0:C_0603_1608Metric, F.Cu at (63.0, 36.7)
- added C2: 1u, NONIK0:C_0603_1608Metric, B.Cu at (70.4, 26.3)
- added C3: 10u, NONIK0:C_0603_1608Metric, B.Cu at (70.4, 33.0)
- added U3: AP3602A, NONIK0:SOT-23-6, B.Cu at (70.4, 29.7)
- moved R2 24.4 mm to (48.6, 16.7)
Connections:
- U1 pad 10: VCC -> Vled
- U1 pad 3: VCC -> Vled
Routing:
- net VCC: track 160.1 -> 103.8 mm, vias 1 -> 0
- net GND: track 250.5 -> 227.0 mm
- net Vled: track 0.00 -> 21.2 mm
- net SCL: track 61.6 -> 50.8 mm, vias 1 -> 0

Commit message: pcb done, pending review
Parts:
- added JP1: SolderJumper_2_Bridged, NONIK0:SolderJumper-2_P1.3mm_Bridged_RoundedPad1.0x1.5mm, B.Cu at (70.9, 32.4)
- C1: moved to B.Cu
- moved C1 12.5 mm to (70.4, 26.7)
- moved R2 5.57 mm to (52.5, 20.6), turned to 90 degrees
- moved C3 4.64 mm to (67.6, 29.3), turned to -90 degrees
- moved C2 4.09 mm to (73.1, 29.3), turned to 90 degrees
- moved BZ1 0.63 mm to (49.7, 20.5)
- moved U3 0.38 mm to (70.4, 29.3)
Routing:
- net VCC: track 103.8 -> 148.3 mm, vias 0 -> 2
- net Vled: track 21.2 -> 59.9 mm
- net BUZZ: track 38.3 -> 59.7 mm
- net RESET: track 52.1 -> 71.1 mm
- net SCL: track 50.8 -> 61.3 mm, vias 0 -> 1
- net GND: track 227.0 -> 235.3 mm, vias 0 -> 1
- net Net-(BZ1-+): track 0.00 -> 5.33 mm
- net UPDI: track 59.6 -> 62.0 mm
- net CE: track 30.8 -> 28.8 mm
- net Net-(U3-C-): track 0.00 -> 1.95 mm
- net Net-(U3-C+): track 0.00 -> 1.69 mm

Commit message: fit and finish things
Parts:
- J1: value AVR-UPDI-6 -> AVR-UPDI-3
- U1: value HCMS-291X -> LED_HCMS-2915
- moved JP1 0.25 mm to (71.2, 32.4)
Routing:
- net GND: track 235.3 -> 251.1 mm, vias 1 -> 2
- net CE: track 28.8 -> 28.1 mm
